Commit message: Update code

File: src/agv0509test6/urdf/agv0509test6.urdf (robot description, URDF)
Before this commit: robot agv0509test6, 6 links, 5 joints
Links:
- added link imu_link, mass 0.01; visual box size=0.02 0.02 0.02
Joints:
- added joint imu_joint: type fixed, parent Base_Link, child imu_link, origin xyz=0 0 0.05 rpy=0 0 0
- joint Left_Wheel_jt: type continuous -> fixed
- joint Lidar_jt: origin xyz=0.3305 -0.015607 0.094 rpy=0 0 0 -> xyz=0.3305 -0.015607 0.094 rpy=0 0 3.14159265
- joint Right_Wheel_jt: type continuous -> fixed

File: src/agv_description/urdf/agv0509test6.urdf (robot description, URDF)
Before this commit: robot agv0509test6, 6 links, 5 joints
Links:
- added link imu_link, mass 0.01; visual box size=0.02 0.02 0.02
- link Base_Link: geometry collision mesh filename=package://agv0509test6/meshes/Base_Link.stl; visual mesh filename=package://agv0509test6/meshes/Base_Link.stl
- link Base_footprint: geometry collision mesh filename=package://agv0509test6/meshes/Base_footprint.stl; visual mesh filename=package://agv0509test6/meshes/Base_footprint.stl
- link Left_Wheel: geometry collision mesh filename=package://agv0509test6/meshes/Left_Wheel.stl; visual mesh filename=package://agv0509test6/meshes/Left_Wheel.stl
- link Lidar: geometry collision mesh filename=package://agv0509test6/meshes/Lidar.stl; visual mesh filename=package://agv0509test6/meshes/Lidar.stl
- link Mam_xoay: geometry collision mesh filename=package://agv0509test6/meshes/Mam_xoay.stl; visual mesh filename=package://agv0509test6/meshes/Mam_xoay.stl
- link Right_Wheel: geometry collision mesh filename=package://agv0509test6/meshes/Right_Wheel.stl; visual mesh filename=package://agv0509test6/meshes/Right_Wheel.stl
Joints:
- added joint imu_joint: type fixed, parent Base_Link, child imu_link, origin xyz=0 0 0.05 rpy=0 0 0
- joint Left_Wheel_jt: type continuous -> fixed
- joint Right_Wheel_jt: type continuous -> fixed
